Commit message: add all robots parts to urdf

File: src/arduinobot_description/urdf/arduinobot.urdf.xacro (robot description, xacro)
@@ -1,8 +1,11 @@
 <?xml version="1.0"?>
 <robot xmlns:xacro="http://www.ros.org/wiki/xacro" name="arduinobot">
+    <xacro:property name="PI" value="3.1459"/>
+    <xacro:property name="effort" value="30.0"/>
+    <xacro:property name="velocity" value="10.0"/>
     <link name="world"/>
-    <link name="basement_link">
+    <link name="base_link">
         <visual>
-            <origin xyz="0.0 0.0 0.0" rpy="0.0 0.0 0.0"/>
+            <origin xyz="-0.5 -0.5 0.0" rpy="0.0 0.0 0.0"/>
             <geometry>
                 <mesh filename="package://arduinobot_description/meshes/basement.STL" scale="0.01 0.01 0.01"/>
@@ -10,8 +13,97 @@
         </visual>
     </link>
-    <joint name="basement_to_world" type="fixed">
+    <joint name="base_to_world" type="fixed">
         <parent link="world"/>
-        <child link="basement_link"/>
+        <child link="base_link"/>
         <origin xyz="0.0 0.0 0.0" rpy="0.0 0.0 0.0"/>
     </joint>
+    <link name="base_plate">
+        <visual>
+            <origin xyz="-0.39 -0.39 -0.56" rpy="0.0 0.0 0.0"/>
+            <geometry>
+                <mesh filename="package://arduinobot_description/meshes/base_plate.STL" scale="0.01 0.01 0.01"/>
+            </geometry>
+        </visual>
+    </link>
+    <joint name="base_plate_to_base" type="revolute">
+        <parent link="base_link"/>
+        <child link="base_plate"/>
+        <origin xyz="0.0 0.0 0.307" rpy="0.0 0.0 0.0"/>
+        <axis xyz="0.0 0.0 1.0"/>
+        <limit lower="-${PI/2}" upper="${PI/2}" effort="${effort}" velocity="${velocity}"/>
+    </joint>
+    <link name="froward_drive_arm">
+        <visual>
+            <origin xyz="0.19 0.06 -0.08" rpy="0.0 -${PI/2} ${PI/2}"/>
+            <geometry>
+                <mesh filename="package://arduinobot_description/meshes/forward_drive_arm.STL" scale="0.01 0.01 0.01"/>
+            </geometry>
+        </visual>
+    </link>
+    <joint name="froward_drive_arm_to_base_plate" type="revolute">
+        <parent link="base_plate"/>
+        <child link="froward_drive_arm"/>
+        <origin xyz="-0.02 0.0 0.35" rpy="0.0 0.0 0.0"/>
+        <axis xyz="1.0 0.0 0.0"/>
+        <limit lower="-${PI/2}" upper="${PI/2}" effort="${effort}" velocity="${velocity}"/>
+    </joint>
+    <link name="horizontal_arm">
+        <visual>
+            <origin xyz="-0.03 -0.4 -0.06" rpy="${PI/2} 0.0 ${PI/2}"/>
+            <geometry>
+                <mesh filename="package://arduinobot_description/meshes/horizontal_arm.STL" scale="0.01 0.01 0.01"/>
+            </geometry>
+        </visual>
+    </link>
+    <joint name="horizontal_arm_to_froward_drive_arm" type="revolute">
+        <parent link="froward_drive_arm"/>
+        <child link="horizontal_arm"/>
+        <origin xyz="0.0 0.0 0.8" rpy="0.0 0.0 0.0"/>
+        <axis xyz="1.0 0.0 0.0"/>
+        <limit lower="-${PI/2}" upper="${PI/2}" effort="${effort}" velocity="${velocity}"/>
+    </joint>
+    <link name="claw_support">
+        <visual>
+            <origin xyz="0.0 -0.05 -0.15" rpy="0.0 0.0 ${PI/2}"/>
+            <geometry>
+                <mesh filename="package://arduinobot_description/meshes/claw_support.STL" scale="0.01 0.01 0.01"/>
+            </geometry>
+        </visual>
+    </link>
+    <joint name="claw_support_to_horizontal_arm" type="fixed">
+        <parent link="horizontal_arm"/>
+        <child link="claw_support"/>
+        <origin xyz="0.0 0.82 0.0" rpy="0.0 0.0 0.0"/>
+    </joint>
+    <link name="right_finger">
+        <visual>
+            <origin xyz="-0.1 0.5 -0.1" rpy="0.0 0.0 -${PI/2}"/>
+            <geometry>
+                <mesh filename="package://arduinobot_description/meshes/right_finger.STL" scale="0.01 0.01 0.01"/>
+            </geometry>
+        </visual>
+    </link>
+    <joint name="right_finger_to_claw_support" type="revolute">
+        <parent link="claw_support"/>
+        <child link="right_finger"/>
+        <origin xyz="-0.04 0.13 -0.1" rpy="0.0 0.0 0.0"/>
+        <axis xyz="-0.0 0.0 1.0"/>
+        <limit lower="-${PI/2}" upper="0" effort="${effort}" velocity="${velocity}"/>
+    </joint>
+    <link name="left_finger">
+        <visual>
+            <origin xyz="-0.04 0.5 -0.1" rpy="0.0 0.0 -${PI/2}"/>
+            <geometry>
+                <mesh filename="package://arduinobot_description/meshes/left_finger.STL" scale="0.01 0.01 0.01"/>
+            </geometry>
+        </visual>
+    </link>
+    <joint name="left_finger_to_claw_support" type="revolute">
+        <parent link="claw_support"/>
+        <child link="left_finger"/>
+        <origin xyz="-0.22 0.13 -0.1" rpy="0.0 0.0 0.0"/>
+        <axis xyz="0.0 0.0 1.0"/>
+        <mimic joint="right_finger_to_claw_support" multiplier="-1"/>
+        <limit lower="0.0" upper="${PI/2}" effort="${effort}" velocity="${velocity}"/>
+    </joint>
 </robot>

Commit message: add gazebo sim

File: src/arduinobot_description/urdf/arduinobot.urdf.xacro (robot description, xacro)
@@ -4,6 +4,15 @@
     <xacro:property name="effort" value="30.0"/>
     <xacro:property name="velocity" value="10.0"/>
+    <xacro:macro name="default_inertial" params="mass">
+        <inertial>
+            <mass value="${mass}"/>
+            <inertia ixx="1.0" ixy="0.0" ixz="0.0"
+                     iyy="1.0" iyz="0.0"
+                     izz="1.0" />
+        </inertial>
+    </xacro:macro>
     <link name="world"/>
     <link name="base_link">
+        <xacro:default_inertial mass="1.0"/>
         <visual>
             <origin xyz="-0.5 -0.5 0.0" rpy="0.0 0.0 0.0"/>
@@ -12,4 +21,10 @@
             </geometry>
         </visual>
+        <collision>
+            <origin xyz="-0.5 -0.5 0.0" rpy="0.0 0.0 0.0"/>
+            <geometry>
+                <mesh filename="package://arduinobot_description/meshes/basement.STL" scale="0.01 0.01 0.01"/>
+            </geometry>
+        </collision>
     </link>
     <joint name="base_to_world" type="fixed">
@@ -19,4 +34,5 @@
     </joint>
     <link name="base_plate">
+        <xacro:default_inertial mass="0.1"/>
         <visual>
             <origin xyz="-0.39 -0.39 -0.56" rpy="0.0 0.0 0.0"/>
@@ -25,4 +41,10 @@
             </geometry>
         </visual>
+        <collision>
+            <origin xyz="-0.39 -0.39 -0.56" rpy="0.0 0.0 0.0"/>
+            <geometry>
+                <mesh filename="package://arduinobot_description/meshes/base_plate.STL" scale="0.01 0.01 0.01"/>
+            </geometry>
+        </collision>
     </link>
     <joint name="base_plate_to_base" type="revolute">
@@ -34,4 +56,5 @@
     </joint>
     <link name="froward_drive_arm">
+        <xacro:default_inertial mass="0.1"/>
         <visual>
             <origin xyz="0.19 0.06 -0.08" rpy="0.0 -${PI/2} ${PI/2}"/>
@@ -40,4 +63,10 @@
             </geometry>
         </visual>
+        <collision>
+            <origin xyz="0.19 0.06 -0.08" rpy="0.0 -${PI/2} ${PI/2}"/>
+            <geometry>
+                <mesh filename="package://arduinobot_description/meshes/forward_drive_arm.STL" scale="0.01 0.01 0.01"/>
+            </geometry>
+        </collision>
     </link>
     <joint name="froward_drive_arm_to_base_plate" type="revolute">
@@ -49,4 +78,5 @@
     </joint>
     <link name="horizontal_arm">
+        <xacro:default_inertial mass="0.1"/>
         <visual>
             <origin xyz="-0.03 -0.4 -0.06" rpy="${PI/2} 0.0 ${PI/2}"/>
@@ -55,4 +85,10 @@
             </geometry>
         </visual>
+        <collision>
+            <origin xyz="-0.03 -0.4 -0.06" rpy="${PI/2} 0.0 ${PI/2}"/>
+            <geometry>
+                <mesh filename="package://arduinobot_description/meshes/horizontal_arm.STL" scale="0.01 0.01 0.01"/>
+            </geometry>
+        </collision>
     </link>
     <joint name="horizontal_arm_to_froward_drive_arm" type="revolute">
@@ -64,4 +100,5 @@
     </joint>
     <link name="claw_support">
+        <xacro:default_inertial mass="0.05"/>
         <visual>
             <origin xyz="0.0 -0.05 -0.15" rpy="0.0 0.0 ${PI/2}"/>
@@ -70,4 +107,10 @@
             </geometry>
         </visual>
+        <collision>
+            <origin xyz="0.0 -0.05 -0.15" rpy="0.0 0.0 ${PI/2}"/>
+            <geometry>
+                <mesh filename="package://arduinobot_description/meshes/claw_support.STL" scale="0.01 0.01 0.01"/>
+            </geometry>
+        </collision>
     </link>
     <joint name="claw_support_to_horizontal_arm" type="fixed">
@@ -77,4 +120,5 @@
     </joint>
     <link name="right_finger">
+        <xacro:default_inertial mass="0.01"/>
         <visual>
             <origin xyz="-0.1 0.5 -0.1" rpy="0.0 0.0 -${PI/2}"/>
@@ -83,4 +127,10 @@
             </geometry>
         </visual>
+        <collision>
+            <origin xyz="-0.1 0.5 -0.1" rpy="0.0 0.0 -${PI/2}"/>
+            <geometry>
+                <mesh filename="package://arduinobot_description/meshes/right_finger.STL" scale="0.01 0.01 0.01"/>
+            </geometry>
+        </collision>
     </link>
     <joint name="right_finger_to_claw_support" type="revolute">
@@ -92,4 +142,5 @@
     </joint>
     <link name="left_finger">
+        <xacro:default_inertial mass="0.01"/>
         <visual>
             <origin xyz="-0.04 0.5 -0.1" rpy="0.0 0.0 -${PI/2}"/>
@@ -98,4 +149,10 @@
             </geometry>
         </visual>
+        <collision>
+            <origin xyz="-0.04 0.5 -0.1" rpy="0.0 0.0 -${PI/2}"/>
+            <geometry>
+                <mesh filename="package://arduinobot_description/meshes/left_finger.STL" scale="0.01 0.01 0.01"/>
+            </geometry>
+        </collision>
     </link>
     <joint name="left_finger_to_claw_support" type="revolute">

Commit message: add controllers

File: src/arduinobot_description/urdf/arduinobot.urdf.xacro (robot description, xacro)
@@ -1,5 +1,8 @@
 <?xml version="1.0"?>
 <robot xmlns:xacro="http://www.ros.org/wiki/xacro" name="arduinobot">
-    <xacro:property name="PI" value="3.1459"/>
+    <xacro:arg name="is_ignition" default="true"/>
+    <xacro:include filename="$(find arduinobot_description)/urdf/arduinobot_gazebo.xacro"/>
+    <xacro:include filename="$(find arduinobot_description)/urdf/arduinobot_ros2_control.xacro"/>
+    <xacro:property name="PI" value="3.14159263359"/>
     <xacro:property name="effort" value="30.0"/>
     <xacro:property name="velocity" value="10.0"/>
